File: hardware/main/supplies.sch (KiCad schematic (older format))
At the start: 7 parts, among them U501 LM7805

Commit message: Abstração do esquemático modificada para separar as duas placas e mostrar a conexão entre elas na folha principal
Changed lines of the file:
@@
 EESchema Schematic File Version 4
 LIBS:main-cache
-EELAYER 26 0
+EELAYER 29 0
 EELAYER END
 $Descr A4 11693 8268
 encoding utf-8
-Sheet 4 8
+Sheet 4 9
 Title ""
 Date ""
@@
 U 1 1 5A007B62
 P 5900 3950
-F 0 "U501" H 5750 4075 50  0000 C CNN
+F 0 "U?" H 5750 4075 50  0000 C CNN
 F 1 "LM7805" H 5900 4100 50  0000 L CNN
 F 2 "KicadZeniteSolarLibrary18:TO-220-3_Horizontal_TabDown_SMD" H 5900 4175 50  0001 C CIN
@@
 U 1 1 5A008895
 P 4900 4400
-F 0 "C501" H 4910 4470 50  0000 L CNN
+F 0 "C?" H 4910 4470 50  0000 L CNN
 F 1 "1uF" H 4910 4320 50  0000 L CNN
 F 2 "Capacitor_Tantalum_SMD:CP_EIA-6032-20_AVX-F_Pad2.25x2.35mm_HandSolder" H 4900 4400 50  0001 C CNN
@@
 U 1 1 5A00899A
 P 5200 4400
-F 0 "C502" H 5210 4470 50  0000 L CNN
+F 0 "C?" H 5210 4470 50  0000 L CNN
 F 1 "100nF" H 5210 4320 50  0000 L CNN
 F 2 "Capacitor_SMD:C_0805_2012Metric_Pad1.15x1.40mm_HandSolder" H 5200 4400 50  0001 C CNN
@@
 U 1 1 5A009BD5
 P 4450 3950
-F 0 "D501" H 4450 4050 50  0000 C CNN
+F 0 "D?" H 4450 4050 50  0000 C CNN
 F 1 "LL4148" H 4450 3850 50  0000 C CNN
 F 2 "Diode_SMD:D_MiniMELF_Handsoldering" H 4450 3775 50  0001 C CNN
@@
 U 1 1 5A00B18A
 P 6500 4400
-F 0 "C503" H 6510 4470 50  0000 L CNN
+F 0 "C?" H 6510 4470 50  0000 L CNN
 F 1 "100nF" H 6510 4320 50  0000 L CNN
 F 2 "Capacitor_SMD:C_0805_2012Metric_Pad1.15x1.40mm_HandSolder" H 6500 4400 50  0001 C CNN
@@
 U 1 1 5AAD0D5C
 P 6850 4400
-F 0 "C504" H 6860 4470 50  0000 L CNN
+F 0 "C?" H 6860 4470 50  0000 L CNN
 F 1 "1uF" H 6860 4320 50  0000 L CNN
 F 2 "Capacitor_Tantalum_SMD:CP_EIA-6032-20_AVX-F_Pad2.25x2.35mm_HandSolder" H 6850 4400 50  0001 C CNN
@@
 U 1 1 5AB12173
 P 4750 3950
-F 0 "F501" H 4750 3890 50  0000 C CNN
+F 0 "F?" H 4750 3890 50  0000 C CNN
 F 1 "500mA" H 4750 4010 50  0000 C CNN
 F 2 "Fuse:Fuse_1206_3216Metric_Pad1.42x1.75mm_HandSolder" H 4750 3950 50  0001 C CNN
@@
 U 1 1 5BE75359
 P 5200 3450
-F 0 "#FLG0501" H 5200 3525 50  0001 C CNN
+F 0 "#FLG?" H 5200 3525 50  0001 C CNN
 F 1 "PWR_FLAG" H 5200 3650 50  0000 C CNN
 F 2 "" H 5200 3450 50  0001 C CNN
@@
 U 1 1 5BE753AF
 P 5200 4900
-F 0 "#FLG0502" H 5200 4975 50  0001 C CNN
+F 0 "#FLG?" H 5200 4975 50  0001 C CNN
 F 1 "PWR_FLAG" H 5200 5100 50  0000 C CNN
 F 2 "" H 5200 4900 50  0001 C CNN

Commit message: TO-DO List criada na folha principal
Changed lines of the file:
@@
 $Descr A4 11693 8268
 encoding utf-8
-Sheet 4 9
+Sheet 6 9
 Title ""
 Date ""
@@
 U 1 1 5A007B62
 P 5900 3950
-F 0 "U?" H 5750 4075 50  0000 C CNN
+AR Path="/5AACFFEF/5A007B62" Ref="U501"  Part="1"
+AR Path="/5CA4DC1F/5CA5A5C0/5A007B62" Ref="U601"  Part="1"
+F 0 "U601" H 5750 4075 50  0000 C CNN
 F 1 "LM7805" H 5900 4100 50  0000 L CNN
 F 2 "KicadZeniteSolarLibrary18:TO-220-3_Horizontal_TabDown_SMD" H 5900 4175 50  0001 C CIN
@@
 U 1 1 5A008895
 P 4900 4400
-F 0 "C?" H 4910 4470 50  0000 L CNN
+AR Path="/5AACFFEF/5A008895" Ref="C501"  Part="1"
+AR Path="/5CA4DC1F/5CA5A5C0/5A008895" Ref="C601"  Part="1"
+F 0 "C601" H 4910 4470 50  0000 L CNN
 F 1 "1uF" H 4910 4320 50  0000 L CNN
 F 2 "Capacitor_Tantalum_SMD:CP_EIA-6032-20_AVX-F_Pad2.25x2.35mm_HandSolder" H 4900 4400 50  0001 C CNN
@@
 U 1 1 5A00899A
 P 5200 4400
-F 0 "C?" H 5210 4470 50  0000 L CNN
+AR Path="/5AACFFEF/5A00899A" Ref="C502"  Part="1"
+AR Path="/5CA4DC1F/5CA5A5C0/5A00899A" Ref="C602"  Part="1"
+F 0 "C602" H 5210 4470 50  0000 L CNN
 F 1 "100nF" H 5210 4320 50  0000 L CNN
 F 2 "Capacitor_SMD:C_0805_2012Metric_Pad1.15x1.40mm_HandSolder" H 5200 4400 50  0001 C CNN
@@
 U 1 1 5A009BD5
 P 4450 3950
-F 0 "D?" H 4450 4050 50  0000 C CNN
+AR Path="/5AACFFEF/5A009BD5" Ref="D501"  Part="1"
+AR Path="/5CA4DC1F/5CA5A5C0/5A009BD5" Ref="D601"  Part="1"
+F 0 "D601" H 4450 4050 50  0000 C CNN
 F 1 "LL4148" H 4450 3850 50  0000 C CNN
 F 2 "Diode_SMD:D_MiniMELF_Handsoldering" H 4450 3775 50  0001 C CNN
@@
 U 1 1 5A00B18A
 P 6500 4400
-F 0 "C?" H 6510 4470 50  0000 L CNN
+AR Path="/5AACFFEF/5A00B18A" Ref="C503"  Part="1"
+AR Path="/5CA4DC1F/5CA5A5C0/5A00B18A" Ref="C603"  Part="1"
+F 0 "C603" H 6510 4470 50  0000 L CNN
 F 1 "100nF" H 6510 4320 50  0000 L CNN
 F 2 "Capacitor_SMD:C_0805_2012Metric_Pad1.15x1.40mm_HandSolder" H 6500 4400 50  0001 C CNN
@@
 U 1 1 5AAD0D5C
 P 6850 4400
-F 0 "C?" H 6860 4470 50  0000 L CNN
+AR Path="/5AACFFEF/5AAD0D5C" Ref="C504"  Part="1"
+AR Path="/5CA4DC1F/5CA5A5C0/5AAD0D5C" Ref="C604"  Part="1"
+F 0 "C604" H 6860 4470 50  0000 L CNN
 F 1 "1uF" H 6860 4320 50  0000 L CNN
 F 2 "Capacitor_Tantalum_SMD:CP_EIA-6032-20_AVX-F_Pad2.25x2.35mm_HandSolder" H 6850 4400 50  0001 C CNN
@@
 U 1 1 5AB12173
 P 4750 3950
-F 0 "F?" H 4750 3890 50  0000 C CNN
+AR Path="/5AACFFEF/5AB12173" Ref="F501"  Part="1"
+AR Path="/5CA4DC1F/5CA5A5C0/5AB12173" Ref="F601"  Part="1"
+F 0 "F601" H 4750 3890 50  0000 C CNN
 F 1 "500mA" H 4750 4010 50  0000 C CNN
 F 2 "Fuse:Fuse_1206_3216Metric_Pad1.42x1.75mm_HandSolder" H 4750 3950 50  0001 C CNN
@@
 U 1 1 5BE75359
 P 5200 3450
-F 0 "#FLG?" H 5200 3525 50  0001 C CNN
+AR Path="/5AACFFEF/5BE75359" Ref="#FLG0501"  Part="1"
+AR Path="/5CA4DC1F/5CA5A5C0/5BE75359" Ref="#FLG0101"  Part="1"
+F 0 "#FLG0101" H 5200 3525 50  0001 C CNN
 F 1 "PWR_FLAG" H 5200 3650 50  0000 C CNN
 F 2 "" H 5200 3450 50  0001 C CNN
@@
 U 1 1 5BE753AF
 P 5200 4900
-F 0 "#FLG?" H 5200 4975 50  0001 C CNN
+AR Path="/5AACFFEF/5BE753AF" Ref="#FLG0502"  Part="1"
+AR Path="/5CA4DC1F/5CA5A5C0/5BE753AF" Ref="#FLG0102"  Part="1"
+F 0 "#FLG0102" H 5200 4975 50  0001 C CNN
 F 1 "PWR_FLAG" H 5200 5100 50  0000 C CNN
 F 2 "" H 5200 4900 50  0001 C CNN

Commit message: Analog passado para o Charger
Changed lines of the file:
@@
 L power:PWR_FLAG #FLG0501
 U 1 1 5BE75359
-P 5200 3450
+P 5200 3850
 AR Path="/5AACFFEF/5BE75359" Ref="#FLG0501"  Part="1"
 AR Path="/5CA4DC1F/5CA5A5C0/5BE75359" Ref="#FLG0101"  Part="1"
-F 0 "#FLG0101" H 5200 3525 50  0001 C CNN
-F 1 "PWR_FLAG" H 5200 3650 50  0000 C CNN
-F 2 "" H 5200 3450 50  0001 C CNN
-F 3 "~" H 5200 3450 50  0001 C CNN
-	1    5200 3450
+F 0 "#FLG0101" H 5200 3925 50  0001 C CNN
+F 1 "PWR_FLAG" H 5200 4050 50  0000 C CNN
+F 2 "" H 5200 3850 50  0001 C CNN
+F 3 "~" H 5200 3850 50  0001 C CNN
+	1    5200 3850
 	1    0    0    -1
 $EndComp
@@
 $EndComp
 Wire Wire Line
-	5200 3450 5200 3950
+	5200 3850 5200 3950
 $EndSCHEMATC

Commit message: Footprints
Changed lines of the file:
@@
 U 1 1 5A007B62
 P 5900 3950
-AR Path="/5AACFFEF/5A007B62" Ref="U501"  Part="1"
-AR Path="/5CA4DC1F/5CA5A5C0/5A007B62" Ref="U601"  Part="1"
-F 0 "U601" H 5750 4075 50  0000 C CNN
+F 0 "U501" H 5750 4075 50  0000 C CNN
 F 1 "LM7805" H 5900 4100 50  0000 L CNN
 F 2 "KicadZeniteSolarLibrary18:TO-220-3_Horizontal_TabDown_SMD" H 5900 4175 50  0001 C CIN
@@
 U 1 1 5A008895
 P 4900 4400
-AR Path="/5AACFFEF/5A008895" Ref="C501"  Part="1"
-AR Path="/5CA4DC1F/5CA5A5C0/5A008895" Ref="C601"  Part="1"
-F 0 "C601" H 4910 4470 50  0000 L CNN
+F 0 "C501" H 4910 4470 50  0000 L CNN
 F 1 "1uF" H 4910 4320 50  0000 L CNN
 F 2 "Capacitor_Tantalum_SMD:CP_EIA-6032-20_AVX-F_Pad2.25x2.35mm_HandSolder" H 4900 4400 50  0001 C CNN
@@
 U 1 1 5A00899A
 P 5200 4400
-AR Path="/5AACFFEF/5A00899A" Ref="C502"  Part="1"
-AR Path="/5CA4DC1F/5CA5A5C0/5A00899A" Ref="C602"  Part="1"
-F 0 "C602" H 5210 4470 50  0000 L CNN
+F 0 "C502" H 5210 4470 50  0000 L CNN
 F 1 "100nF" H 5210 4320 50  0000 L CNN
 F 2 "Capacitor_SMD:C_0805_2012Metric_Pad1.15x1.40mm_HandSolder" H 5200 4400 50  0001 C CNN
@@
 U 1 1 5A009BD5
 P 4450 3950
-AR Path="/5AACFFEF/5A009BD5" Ref="D501"  Part="1"
-AR Path="/5CA4DC1F/5CA5A5C0/5A009BD5" Ref="D601"  Part="1"
-F 0 "D601" H 4450 4050 50  0000 C CNN
+F 0 "D501" H 4450 4050 50  0000 C CNN
 F 1 "LL4148" H 4450 3850 50  0000 C CNN
 F 2 "Diode_SMD:D_MiniMELF_Handsoldering" H 4450 3775 50  0001 C CNN
@@
 U 1 1 5A00B18A
 P 6500 4400
-AR Path="/5AACFFEF/5A00B18A" Ref="C503"  Part="1"
-AR Path="/5CA4DC1F/5CA5A5C0/5A00B18A" Ref="C603"  Part="1"
-F 0 "C603" H 6510 4470 50  0000 L CNN
+F 0 "C503" H 6510 4470 50  0000 L CNN
 F 1 "100nF" H 6510 4320 50  0000 L CNN
 F 2 "Capacitor_SMD:C_0805_2012Metric_Pad1.15x1.40mm_HandSolder" H 6500 4400 50  0001 C CNN
@@
 U 1 1 5AAD0D5C
 P 6850 4400
-AR Path="/5AACFFEF/5AAD0D5C" Ref="C504"  Part="1"
-AR Path="/5CA4DC1F/5CA5A5C0/5AAD0D5C" Ref="C604"  Part="1"
-F 0 "C604" H 6860 4470 50  0000 L CNN
+F 0 "C504" H 6860 4470 50  0000 L CNN
 F 1 "1uF" H 6860 4320 50  0000 L CNN
 F 2 "Capacitor_Tantalum_SMD:CP_EIA-6032-20_AVX-F_Pad2.25x2.35mm_HandSolder" H 6850 4400 50  0001 C CNN
@@
 U 1 1 5AB12173
 P 4750 3950
-AR Path="/5AACFFEF/5AB12173" Ref="F501"  Part="1"
-AR Path="/5CA4DC1F/5CA5A5C0/5AB12173" Ref="F601"  Part="1"
-F 0 "F601" H 4750 3890 50  0000 C CNN
+F 0 "F501" H 4750 3890 50  0000 C CNN
 F 1 "500mA" H 4750 4010 50  0000 C CNN
 F 2 "Fuse:Fuse_1206_3216Metric_Pad1.42x1.75mm_HandSolder" H 4750 3950 50  0001 C CNN
@@
 L power:PWR_FLAG #FLG0501
 U 1 1 5BE75359
-P 5200 3850
-AR Path="/5AACFFEF/5BE75359" Ref="#FLG0501"  Part="1"
-AR Path="/5CA4DC1F/5CA5A5C0/5BE75359" Ref="#FLG0101"  Part="1"
-F 0 "#FLG0101" H 5200 3925 50  0001 C CNN
-F 1 "PWR_FLAG" H 5200 4050 50  0000 C CNN
-F 2 "" H 5200 3850 50  0001 C CNN
-F 3 "~" H 5200 3850 50  0001 C CNN
-	1    5200 3850
+P 5200 3450
+F 0 "#FLG0501" H 5200 3525 50  0001 C CNN
+F 1 "PWR_FLAG" H 5200 3650 50  0000 C CNN
+F 2 "" H 5200 3450 50  0001 C CNN
+F 3 "~" H 5200 3450 50  0001 C CNN
+	1    5200 3450
 	1    0    0    -1
 $EndComp
@@
 U 1 1 5BE753AF
 P 5200 4900
-AR Path="/5AACFFEF/5BE753AF" Ref="#FLG0502"  Part="1"
-AR Path="/5CA4DC1F/5CA5A5C0/5BE753AF" Ref="#FLG0102"  Part="1"
-F 0 "#FLG0102" H 5200 4975 50  0001 C CNN
+F 0 "#FLG0502" H 5200 4975 50  0001 C CNN
 F 1 "PWR_FLAG" H 5200 5100 50  0000 C CNN
 F 2 "" H 5200 4900 50  0001 C CNN
@@
 $EndComp
 Wire Wire Line
-	5200 3850 5200 3950
+	5200 3450 5200 3950
 $EndSCHEMATC
