File: hardware/main/Charger.sch (KiCad schematic (older format))
At the start: 48 parts, among them K1 DIPxx-1Axx-13x, K2 SANYOU_SRD_Form_C, Q1 Q_NPN_BEC, Q2 BCV27, Q3 BCV27

Commit message: CAN CTRL_D / CAN_ON_OFF removidos.
Connections:
- net GND is gone; now on net GNDPWR: C?.2, C?.2, C?.2, C?.2, U?.2 (GND)
Changed lines of the file:
@@
 $Descr A3 16535 11693
 encoding utf-8
-Sheet 2 9
+Sheet 2 8
 Title ""
 Date ""
@@
 Wire Wire Line
 	7700 4900 7700 5250
+$Comp
+L power:GNDPWR #PWR?
+U 1 1 5CB769FE
+P 4050 8600
+F 0 "#PWR?" H 4050 8400 50  0001 C CNN
+F 1 "GNDPWR" H 4054 8446 50  0000 C CNN
+F 2 "" H 4050 8550 50  0001 C CNN
+F 3 "" H 4050 8550 50  0001 C CNN
+	1    4050 8600
+	1    0    0    -1
+$EndComp
+Wire Wire Line
+	4050 8600 4050 8450
 $EndSCHEMATC

Commit message: Novos capacitores anotados
Parts:
- gave numbers to parts that had none: 11
Changed lines of the file:
@@
 U_BAT+
 $Comp
-L Device:CP1_Small C?
+L Device:CP1_Small C204
 U 1 1 5CABA9BC
 P 4150 5250
-F 0 "C?" H 4250 5300 50  0000 L CNN
+F 0 "C204" H 4250 5300 50  0000 L CNN
 F 1 "4700u" H 4250 5250 50  0000 L CNN
 F 2 "" H 4150 5250 50  0001 C CNN
@@
 	4150 5350 4150 5450
 $Comp
-L power:GNDPWR #PWR?
+L power:GNDPWR #PWR0110
 U 1 1 5CAC48B2
 P 4150 5500
-F 0 "#PWR?" H 4150 5300 50  0001 C CNN
+F 0 "#PWR0110" H 4150 5300 50  0001 C CNN
 F 1 "GNDPWR" H 4154 5346 50  0000 C CNN
 F 2 "" H 4150 5450 50  0001 C CNN
@@
 $EndComp
 $Comp
-L Device:C_Small C?
+L Device:C_Small C203
 U 1 1 5CAC7DC0
 P 3950 5250
-F 0 "C?" H 4042 5296 50  0000 L CNN
+F 0 "C203" H 4042 5296 50  0000 L CNN
 F 1 "100n" H 4042 5205 50  0000 L CNN
 F 2 "" H 3950 5250 50  0001 C CNN
@@
 +12V
 $Comp
-L Device:C_Small C?
+L Device:C_Small C201
 U 1 1 5CADFEC7
 P 2600 2950
-F 0 "C?" H 2692 2996 50  0000 L CNN
+F 0 "C201" H 2692 2996 50  0000 L CNN
 F 1 "100n" H 2692 2905 50  0000 L CNN
 F 2 "" H 2600 2950 50  0001 C CNN
@@
 Connection ~ 2400 2950
 $Comp
-L Device:C_Small C?
+L Device:C_Small C202
 U 1 1 5CAF15BA
 P 3100 2950
-F 0 "C?" H 3192 2996 50  0000 L CNN
+F 0 "C202" H 3192 2996 50  0000 L CNN
 F 1 "100n" H 3192 2905 50  0000 L CNN
 F 2 "" H 3100 2950 50  0001 C CNN
@@
 AR Path="/5AACFFEF/5CB0F970" Ref="U?"  Part="1"
 AR Path="/5CA4DC1F/5CA5A5C0/5CB0F970" Ref="U?"  Part="1"
-AR Path="/5C9C4D6B/5CB0F970" Ref="U?"  Part="1"
-F 0 "U?" H 3300 7725 50  0000 C CNN
+AR Path="/5C9C4D6B/5CB0F970" Ref="U201"  Part="1"
+F 0 "U201" H 3300 7725 50  0000 C CNN
 F 1 "LM7812" H 3450 7750 50  0000 L CNN
 F 2 "KicadZeniteSolarLibrary18:TO-220-3_Horizontal_TabDown_SMD" H 3450 7825 50  0001 C CIN
@@
 AR Path="/5AACFFEF/5CB0F97E" Ref="C?"  Part="1"
 AR Path="/5CA4DC1F/5CA5A5C0/5CB0F97E" Ref="C?"  Part="1"
-AR Path="/5C9C4D6B/5CB0F97E" Ref="C?"  Part="1"
-F 0 "C?" H 2760 8120 50  0000 L CNN
+AR Path="/5C9C4D6B/5CB0F97E" Ref="C206"  Part="1"
+F 0 "C206" H 2760 8120 50  0000 L CNN
 F 1 "100nF" H 2760 7970 50  0000 L CNN
 F 2 "Capacitor_SMD:C_0805_2012Metric_Pad1.15x1.40mm_HandSolder" H 2750 8050 50  0001 C CNN
@@
 AR Path="/5AACFFEF/5CB0F984" Ref="D?"  Part="1"
 AR Path="/5CA4DC1F/5CA5A5C0/5CB0F984" Ref="D?"  Part="1"
-AR Path="/5C9C4D6B/5CB0F984" Ref="D?"  Part="1"
-F 0 "D?" H 1800 7700 50  0000 C CNN
+AR Path="/5C9C4D6B/5CB0F984" Ref="D201"  Part="1"
+F 0 "D201" H 1800 7700 50  0000 C CNN
 F 1 "LL4148" H 1800 7500 50  0000 C CNN
 F 2 "Diode_SMD:D_MiniMELF_Handsoldering" H 1800 7425 50  0001 C CNN
@@
 AR Path="/5AACFFEF/5CB0F98B" Ref="C?"  Part="1"
 AR Path="/5CA4DC1F/5CA5A5C0/5CB0F98B" Ref="C?"  Part="1"
-AR Path="/5C9C4D6B/5CB0F98B" Ref="C?"  Part="1"
-F 0 "C?" H 4060 8120 50  0000 L CNN
+AR Path="/5C9C4D6B/5CB0F98B" Ref="C207"  Part="1"
+F 0 "C207" H 4060 8120 50  0000 L CNN
 F 1 "100nF" H 4060 7970 50  0000 L CNN
 F 2 "Capacitor_SMD:C_0805_2012Metric_Pad1.15x1.40mm_HandSolder" H 4050 8050 50  0001 C CNN
@@
 AR Path="/5AACFFEF/5CB0F997" Ref="F?"  Part="1"
 AR Path="/5CA4DC1F/5CA5A5C0/5CB0F997" Ref="F?"  Part="1"
-AR Path="/5C9C4D6B/5CB0F997" Ref="F?"  Part="1"
-F 0 "F?" H 2100 7540 50  0000 C CNN
+AR Path="/5C9C4D6B/5CB0F997" Ref="F201"  Part="1"
+F 0 "F201" H 2100 7540 50  0000 C CNN
 F 1 "500mA" H 2100 7660 50  0000 C CNN
 F 2 "Fuse:Fuse_1206_3216Metric_Pad1.42x1.75mm_HandSolder" H 2100 7600 50  0001 C CNN
@@
 AR Path="/5AACFFEF/5CB0F9BC" Ref="#FLG?"  Part="1"
 AR Path="/5CA4DC1F/5CA5A5C0/5CB0F9BC" Ref="#FLG?"  Part="1"
-AR Path="/5C9C4D6B/5CB0F9BC" Ref="#FLG?"  Part="1"
-F 0 "#FLG?" H 2750 7575 50  0001 C CNN
+AR Path="/5C9C4D6B/5CB0F9BC" Ref="#FLG0103"  Part="1"
+F 0 "#FLG0103" H 2750 7575 50  0001 C CNN
 F 1 "PWR_FLAG" H 2750 7700 50  0000 C CNN
 F 2 "" H 2750 7500 50  0001 C CNN
@@
 AR Path="/5AACFFEF/5CB0F9C2" Ref="#FLG?"  Part="1"
 AR Path="/5CA4DC1F/5CA5A5C0/5CB0F9C2" Ref="#FLG?"  Part="1"
-AR Path="/5C9C4D6B/5CB0F9C2" Ref="#FLG?"  Part="1"
-F 0 "#FLG?" H 2750 8625 50  0001 C CNN
+AR Path="/5C9C4D6B/5CB0F9C2" Ref="#FLG0104"  Part="1"
+F 0 "#FLG0104" H 2750 8625 50  0001 C CNN
 F 1 "PWR_FLAG" H 2750 8750 50  0000 C CNN
 F 2 "" H 2750 8550 50  0001 C CNN
@@
 AR Path="/5AACFFEF/5CB0F978" Ref="C?"  Part="1"
 AR Path="/5CA4DC1F/5CA5A5C0/5CB0F978" Ref="C?"  Part="1"
-AR Path="/5C9C4D6B/5CB0F978" Ref="C?"  Part="1"
-F 0 "C?" H 2460 8120 50  0000 L CNN
+AR Path="/5C9C4D6B/5CB0F978" Ref="C205"  Part="1"
+F 0 "C205" H 2460 8120 50  0000 L CNN
 F 1 "1uF" H 2460 7970 50  0000 L CNN
 F 2 "Capacitor_Tantalum_SMD:CP_EIA-6032-20_AVX-F_Pad2.25x2.35mm_HandSolder" H 2450 8050 50  0001 C CNN
@@
 AR Path="/5AACFFEF/5CB0F991" Ref="C?"  Part="1"
 AR Path="/5CA4DC1F/5CA5A5C0/5CB0F991" Ref="C?"  Part="1"
-AR Path="/5C9C4D6B/5CB0F991" Ref="C?"  Part="1"
-F 0 "C?" H 4410 8120 50  0000 L CNN
+AR Path="/5C9C4D6B/5CB0F991" Ref="C208"  Part="1"
+F 0 "C208" H 4410 8120 50  0000 L CNN
 F 1 "1uF" H 4410 7970 50  0000 L CNN
 F 2 "Capacitor_Tantalum_SMD:CP_EIA-6032-20_AVX-F_Pad2.25x2.35mm_HandSolder" H 4400 8050 50  0001 C CNN
@@
 	7700 4900 7700 5250
 $Comp
-L power:GNDPWR #PWR?
+L power:GNDPWR #PWR0111
 U 1 1 5CB769FE
 P 4050 8600
-F 0 "#PWR?" H 4050 8400 50  0001 C CNN
+F 0 "#PWR0111" H 4050 8400 50  0001 C CNN
 F 1 "GNDPWR" H 4054 8446 50  0000 C CNN
 F 2 "" H 4050 8550 50  0001 C CNN

Commit message: Analog passado para o Charger
Parts:
- added JP201, JP202, JP203: Jp_TEST, symbol Device:Jumper_NC_Small
- added NT201: Net-Tie_2, symbol Device:Net-Tie_2
Connections:
- net +BAT is gone; now on net U_BAT+: K2.1
- net +CAP: now also JP203.1
- net GNDPWR: now also NT201.2
- net U_BAT+: now also JP202.1
- new net +5V: JP201.1
- new net GNDA: NT201.1
- new net sheet5CBAED96/+5V: JP201.2
- new net sheet5CBAED96/in1+: JP202.2
- new net sheet5CBAED96/in2+: JP203.2

Commit message: Esquematico primeira versão Erro de referencia dos componentes na PCB com os do Esquematico solucionados
Pontos de teste adicionados
Alimentar o analog com +12V
Adicionar Snubber para os reles
Parts:
- added C6: 100n, Capacitor_SMD:C_0805_2012Metric_Pad1.15x1.40mm_HandSolder, symbol Device:C_Small
- added C7: 100n, Capacitor_THT:CP_Radial_D18.0mm_P7.50mm, symbol Device:C_Small
- added D8: GRN_LED, symbol Device:LED
- added R16: 470, symbol Device:R_Small_US
- added R7, R8: 1R, symbol Device:R_Small
- added TP1: RL_ON, TestPoint:TestPoint_Pad_D1.5mm, symbol Connector:TestPoint
- added TP10: TH+, symbol Connector:TestPoint
- added TP11: TH-, symbol Connector:TestPoint
- added TP12: RL_OFF, symbol Connector:TestPoint
- added TP2: Charge, TestPoint:TestPoint_Pad_D1.5mm, symbol Connector:TestPoint
- added TP3: B_CH, TestPoint:TestPoint_Pad_D1.5mm, symbol Connector:TestPoint
- added TP4: B_ON, TestPoint:TestPoint_Pad_D1.5mm, symbol Connector:TestPoint
- added TP5: ON, TestPoint:TestPoint_Pad_D1.5mm, symbol Connector:TestPoint
- added TP6: CH-, symbol Connector:TestPoint
- added TP7: OFF, symbol Connector:TestPoint
- added TP8: CH+, symbol Connector:TestPoint
- added TP9: B_OFF, symbol Connector:TestPoint
- C1: renamed from C2; footprint (none) -> Capacitor_SMD:C_0805_2012Metric_Pad1.15x1.40mm_HandSolder
- C10: renamed from C203; footprint (none) -> Capacitor_SMD:C_0805_2012Metric_Pad1.15x1.40mm_HandSolder
- C12: renamed from C204; footprint (none) -> Capacitor_SMD:C_0805_2012Metric_Pad1.15x1.40mm_HandSolder
- C2: renamed from C1; footprint (none) -> Capacitor_SMD:C_0805_2012Metric_Pad1.15x1.40mm_HandSolder
- C3: renamed from C205; footprint Capacitor_Tantalum_SMD:CP_EIA-6032-20_AVX-F_Pad2.25x2.35mm_HandSolder -> Capacitor_SMD:C_0805_2012Metric_Pad1.15x1.40mm_HandSolder
- C4: renamed from C201; footprint (none) -> Capacitor_SMD:C_0805_2012Metric_Pad1.15x1.40mm_HandSolder
- C8: renamed from C202; footprint (none) -> Capacitor_SMD:C_0805_2012Metric_Pad1.15x1.40mm_HandSolder
- C9: renamed from C3; footprint (none) -> Capacitor_SMD:C_0805_2012Metric_Pad1.15x1.40mm_HandSolder
- D1: renamed from D201; footprint Diode_SMD:D_MiniMELF_Handsoldering -> Package_TO_SOT_SMD:SOT-23_Handsoldering
- D2: renamed from D1; footprint Diode_SMD:D_MiniMELF -> LED_SMD:LED_0805_2012Metric_Pad1.15x1.40mm_HandSolder
- D4: renamed from D3; footprint Diode_SMD:D_MiniMELF -> LED_SMD:LED_0805_2012Metric_Pad1.15x1.40mm_HandSolder
- D5: renamed from D4; footprint (none) -> Diode_THT:D_DO-201AD_P15.24mm_Horizontal
- D6: renamed from D5; footprint (none) -> LED_SMD:LED_0805_2012Metric_Pad1.15x1.40mm_HandSolder
- F2: renamed from F1; footprint (none) -> KicadZeniteSolarLibrary18:Fuse_Holder_5x20
- K1: footprint Relay_THT:Relay_StandexMeder_DIP_LowProfile -> Relay_THT:Relay_SPDT_SANYOU_SRD_Series_Form_C
- Q2: renamed from Q1; footprint (none) -> Package_TO_SOT_SMD:TSOT-23_HandSoldering
- R1: renamed from R2; footprint (none) -> Resistor_SMD:R_0805_2012Metric_Pad1.15x1.40mm_HandSolder
- R10: renamed from R8; footprint (none) -> Resistor_SMD:R_0805_2012Metric_Pad1.15x1.40mm_HandSolder
- R2: renamed from R1; footprint (none) -> Resistor_SMD:R_0805_2012Metric_Pad1.15x1.40mm_HandSolder
- R3: renamed from R4; footprint (none) -> Resistor_SMD:R_0805_2012Metric_Pad1.15x1.40mm_HandSolder
- R4: renamed from R3; footprint (none) -> Resistor_SMD:R_0805_2012Metric_Pad1.15x1.40mm_HandSolder
- R5: renamed from R6; footprint (none) -> Resistor_SMD:R_0805_2012Metric_Pad1.15x1.40mm_HandSolder
- R6: renamed from R5; footprint (none) -> Resistor_SMD:R_0805_2012Metric_Pad1.15x1.40mm_HandSolder
- R9: renamed from R7; footprint (none) -> Resistor_SMD:R_0805_2012Metric_Pad1.15x1.40mm_HandSolder
- U1: renamed from U201; footprint KicadZeniteSolarLibrary18:TO-220-3_Horizontal_TabDown_SMD -> Package_SO:SOIC-8_3.9x4.9mm_P1.27mm
- renumbered C207 to C11, C208 to C13, C206 to C5, D2 to D3, D6 to D7, F201 to F1, H203 to H1, H3 to H2, H206 to H3, H207 to H4, H201 to H5, H202 to H6, H204 to H7, H205 to H8, JP202 to JP1, JP203 to JP2, JP201 to JP3, NT201 to NT1, Q2 to Q1, R9 to R11, R10 to R12, R11 to R13, R12 to R14, R13 to R15
Connections:
- net +5V is gone; now on net +12V: JP3.1
- net +12V: now also R16.1, TP8.1
- net +CAP: now also C7.1
- net Charge: now also R8.2, TP10.1, TP2.1
- net GNDPWR: now also D8.1 (K)
- net RL_OFF: now also TP12.1
- net RL_ON: now also TP1.1
- net U_BAT+: now also C6.1, R7.2
- net at R12.2, TH1.1: now also TP11.1
- net at K1.2 (NA), R9.1: now also TP7.1
- net at K1.3 (NF), R5.1: now also TP5.1
- net at D3.2 (A), K2.2, R6.1: now also TP6.1
- net at C2.1, Q2.1 (B), R2.1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: now also TP3.1
- net sheet5CBAED96/+5V renamed sheet5CBAED96/+12V
- new net: C7.2, R7.1
- new net: C6.2, R8.1
- new net: D8.2 (A), R16.2
Other:
- moved on the sheet: C1, C4, C8, C9, H1, H2, JP3, K1, NT1, Q1, Q3, R1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

Commit message: Footprints
Parts:
- added H1, H2, H3, H4: MountingHole, MountingHole:MountingHole_3.2mm_M3, symbol Mechanical:MountingHole
- C807: renamed from C7; footprint Capacitor_THT:CP_Radial_D18.0mm_P7.50mm -> Capacitor_SMD:C_0805_2012Metric_Pad1.15x1.40mm_HandSolder
- D801: renamed from D1; footprint Package_TO_SOT_SMD:SOT-23_Handsoldering -> Diode_SMD:D_MiniMELF_Handsoldering
- D802: renamed from D2; footprint LED_SMD:LED_0805_2012Metric_Pad1.15x1.40mm_HandSolder -> Diode_SMD:D_MiniMELF_Handsoldering
- D803: renamed from D3; footprint Diode_SMD:D_MiniMELF -> Diode_SMD:D_MiniMELF_Handsoldering
- D804: renamed from D4; footprint LED_SMD:LED_0805_2012Metric_Pad1.15x1.40mm_HandSolder -> Diode_SMD:D_MiniMELF_Handsoldering
- D805: renamed from D5; footprint Diode_THT:D_DO-201AD_P15.24mm_Horizontal -> LED_SMD:LED_0805_2012Metric_Pad1.15x1.40mm_HandSolder
- D807: renamed from D7; footprint (none) -> LED_SMD:LED_0805_2012Metric_Pad1.15x1.40mm_HandSolder
- D808: renamed from D8; footprint (none) -> LED_SMD:LED_0805_2012Metric_Pad1.15x1.40mm_HandSolder
- F802: renamed from F2; footprint KicadZeniteSolarLibrary18:Fuse_Holder_5x20 -> KicadZeniteSolarLibrary18:MegaFuse
- H801: renamed from H1; footprint (none) -> MountingHole:MountingHole_3.2mm_M3_DIN965_Pad
- H802: renamed from H2; value +CAP -> +BAT; footprint (none) -> MountingHole:MountingHole_3.2mm_M3_DIN965_Pad
- H803: renamed from H3; footprint (none) -> MountingHole:MountingHole_3.2mm_M3_DIN965_Pad
- H804: renamed from H4; footprint (none) -> MountingHole:MountingHole_3.2mm_M3_DIN965_Pad
- JP801: renamed from JP1; footprint (none) -> Resistor_SMD:R_0805_2012Metric_Pad1.15x1.40mm_HandSolder
- JP802: renamed from JP2; footprint (none) -> Resistor_SMD:R_0805_2012Metric_Pad1.15x1.40mm_HandSolder
- JP803: renamed from JP3; footprint (none) -> Resistor_SMD:R_0805_2012Metric_Pad1.15x1.40mm_HandSolder
- K801: renamed from K1; footprint Relay_THT:Relay_SPDT_SANYOU_SRD_Series_Form_C -> KicadZeniteSolarLibrary18:Mega_Relay_K100
- NT801: renamed from NT1; footprint (none) -> Resistor_SMD:R_0805_2012Metric_Pad1.15x1.40mm_HandSolder
- R807: renamed from R7; footprint (none) -> Resistor_SMD:R_0805_2012Metric_Pad1.15x1.40mm_HandSolder
- R808: renamed from R8; footprint (none) -> Resistor_SMD:R_0805_2012Metric_Pad1.15x1.40mm_HandSolder
- R811: renamed from R11; footprint (none) -> Resistor_SMD:R_0805_2012Metric_Pad1.15x1.40mm_HandSolder
- R812: renamed from R12; footprint (none) -> Resistor_THT:R_Axial_Power_L48.0mm_W12.5mm_P55.88mm
- R813: renamed from R13; footprint (none) -> Resistor_SMD:R_0805_2012Metric_Pad1.15x1.40mm_HandSolder
- R814: renamed from R14; footprint (none) -> Resistor_SMD:R_0805_2012Metric_Pad1.15x1.40mm_HandSolder
- R815: renamed from R15; footprint (none) -> Resistor_SMD:R_0805_2012Metric_Pad1.15x1.40mm_HandSolder
- R816: renamed from R16; footprint (none) -> Resistor_SMD:R_0805_2012Metric_Pad1.15x1.40mm_HandSolder
- TH801: renamed from TH1; footprint (none) -> Resistor_THT:R_Axial_DIN0204_L3.6mm_D1.6mm_P7.62mm_Horizontal
- TP806: renamed from TP6; footprint (none) -> TestPoint:TestPoint_Pad_D1.5mm
- TP807: renamed from TP7; footprint (none) -> TestPoint:TestPoint_Pad_D1.5mm
- TP808: renamed from TP8; footprint (none) -> TestPoint:TestPoint_Pad_D1.5mm
- TP809: renamed from TP9; footprint (none) -> TestPoint:TestPoint_Pad_D1.5mm
- TP810: renamed from TP10; footprint (none) -> TestPoint:TestPoint_Pad_D1.5mm
- TP811: renamed from TP11; footprint (none) -> TestPoint:TestPoint_Pad_D1.5mm
- TP812: renamed from TP12; footprint (none) -> TestPoint:TestPoint_Pad_D1.5mm
- renumbered C1 to C801, C2 to C802, C3 to C803, C4 to C804, C5 to C805, C6 to C806, C8 to C808, C9 to C809, C10 to C810, C11 to C811, C12 to C812, C13 to C813, D6 to D806, F1 to F801, H5 to H805, H6 to H806, H7 to H807, H8 to H808, K2 to K802, Q1 to Q801, Q2 to Q802, Q3 to Q803, R1 to R801, R2 to R802, R3 to R803, R4 to R804, R5 to R805, R6 to R806, R9 to R809, R10 to R810, TP1 to TP801, TP2 to TP802, TP3 to TP803, TP4 to TP804, TP5 to TP805, U1 to U801
Connections:
- net +CAP: no longer C807.1, H802.1, K801.5
- net at C801.1, Q801.1 (B), R801.1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: now also TP804.1
- net at C809.1, Q803.1 (B), R810.1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: now also TP809.1
- new net +BAT: C807.1, H802.1, K801.5
Other:
- moved on the sheet: TP804, TP809

Commit message: Generic layout and relay driver
Connections:
- net +BAT is gone; now on net +CAP: C807.1, H802.1, K801.5
- net Charge: no longer K802.3, R808.2, TH801.2, TP810.1
- new net CH: K802.3, R808.2, TH801.2, TP810.1
Changed lines of the file:
@@
 	3950 4450 4000 4450
 Text Label 3600 4450 2    50   ~ 0
-Charge
+CH
 Text Label 4650 4450 0    50   ~ 0
 +CAP
@@
 Wire Wire Line
 	3300 4450 3550 4450
-$Comp
-L Device:Q_NPN_BEC Q802
-U 1 1 5C9E4DF9
-P 2250 5700
-AR Path="/5C9C4D6B/5C9E4DF9" Ref="Q802"  Part="1"
-AR Path="/5CBD2CE3/5C9E4DF9" Ref="Q?"  Part="1"
-F 0 "Q802" H 2441 5746 50  0000 L CNN
-F 1 "Q_NPN_BEC" H 2441 5655 50  0000 L CNN
-F 2 "Package_TO_SOT_SMD:TSOT-23_HandSoldering" H 2450 5800 50  0001 C CNN
-F 3 "~" H 2250 5700 50  0001 C CNN
-	1    2250 5700
-	1    0    0    -1
-$EndComp
 $Comp
 L Device:R_Small_US R806
@@
 	1950 6250 1950 6200
 $Comp
-L Device:Q_NPN_BEC Q801
-U 1 1 5C9E64EB
-P 2250 2600
-AR Path="/5C9C4D6B/5C9E64EB" Ref="Q801"  Part="1"
-AR Path="/5CBD2CE3/5C9E64EB" Ref="Q?"  Part="1"
-F 0 "Q801" H 2441 2646 50  0000 L CNN
-F 1 "BCV27" H 2441 2555 50  0000 L CNN
-F 2 "Package_TO_SOT_SMD:TSOT-23_HandSoldering" H 2450 2700 50  0001 C CNN
-F 3 "~" H 2250 2600 50  0001 C CNN
-	1    2250 2600
-	1    0    0    -1
-$EndComp
-$Comp
 L Device:R_Small_US R805
 U 1 1 5C9E64F1
@@
 	1950 3150 1950 3100
 $Comp
-L Device:Q_NPN_BEC Q803
-U 1 1 5C9E7354
-P 3350 2600
-AR Path="/5C9C4D6B/5C9E7354" Ref="Q803"  Part="1"
-AR Path="/5CBD2CE3/5C9E7354" Ref="Q?"  Part="1"
-F 0 "Q803" H 3541 2646 50  0000 L CNN
-F 1 "BCV27" H 3541 2555 50  0000 L CNN
-F 2 "Package_TO_SOT_SMD:TSOT-23_HandSoldering" H 3550 2700 50  0001 C CNN
-F 3 "~" H 3350 2600 50  0001 C CNN
-	1    3350 2600
-	-1   0    0    -1
-$EndComp
-$Comp
 L Device:R_Small_US R809
 U 1 1 5C9E735A
@@
 Text Label 2350 1400 2    50   ~ 0
 U_BAT+
-Text Label 3250 1400 0    50   ~ 0
-+BAT
 $Comp
 L Mechanical:MountingHole_Pad H802
@@
 	1    0    0    -1
 $EndComp
-Connection ~ 2050 5700
 $Comp
 L Connector:TestPoint TP802
@@
 	1    0    0    -1
 $EndComp
-Connection ~ 2050 2600
 Wire Wire Line
 	1950 2600 2050 2600
-Connection ~ 3550 2600
 Wire Wire Line
 	3750 7600 4050 7600
@@
 	8000 8000 7950 8000
 Connection ~ 7950 8000
+Text Label 3300 1400 0    50   ~ 0
++CAP
+Connection ~ 2050 5700
+$Comp
+L Device:Q_NPN_BEC Q802
+U 1 1 5C9E4DF9
+P 2250 5700
+AR Path="/5C9C4D6B/5C9E4DF9" Ref="Q802"  Part="1"
+AR Path="/5CBD2CE3/5C9E4DF9" Ref="Q?"  Part="1"
+F 0 "Q802" H 2441 5746 50  0000 L CNN
+F 1 "Q_NPN_BEC" H 2441 5655 50  0000 L CNN
+F 2 "Package_TO_SOT_SMD:TSOT-23_HandSoldering" H 2450 5800 50  0001 C CNN
+F 3 "~" H 2250 5700 50  0001 C CNN
+	1    2250 5700
+	1    0    0    -1
+$EndComp
+Connection ~ 3550 2600
+$Comp
+L Device:Q_NPN_BEC Q803
+U 1 1 5C9E7354
+P 3350 2600
+AR Path="/5C9C4D6B/5C9E7354" Ref="Q803"  Part="1"
+AR Path="/5CBD2CE3/5C9E7354" Ref="Q?"  Part="1"
+F 0 "Q803" H 3541 2646 50  0000 L CNN
+F 1 "BCV27" H 3541 2555 50  0000 L CNN
+F 2 "Package_TO_SOT_SMD:TSOT-23_HandSoldering" H 3550 2700 50  0001 C CNN
+F 3 "~" H 3350 2600 50  0001 C CNN
+	1    3350 2600
+	-1   0    0    -1
+$EndComp
+Connection ~ 2050 2600
+$Comp
+L Device:Q_NPN_BEC Q801
+U 1 1 5C9E64EB
+P 2250 2600
+AR Path="/5C9C4D6B/5C9E64EB" Ref="Q801"  Part="1"
+AR Path="/5CBD2CE3/5C9E64EB" Ref="Q?"  Part="1"
+F 0 "Q801" H 2441 2646 50  0000 L CNN
+F 1 "BCV27" H 2441 2555 50  0000 L CNN
+F 2 "Package_TO_SOT_SMD:TSOT-23_HandSoldering" H 2450 2700 50  0001 C CNN
+F 3 "~" H 2250 2600 50  0001 C CNN
+	1    2250 2600
+	1    0    0    -1
+$EndComp
 $EndSCHEMATC
