File: hardware/main/main.kicad_pcb (KiCad board)
At the start: 2 copper layers, 85 parts, among them J1 Screw_Terminal_01x02, J2 Screw_Terminal_01x03, J401 USART, J601 RJ45, J602 RJ45, K1 coil: 12VDC, contact: 125V/10A, Q1 BCV27, U1 4N25, U201 MCP2551-I/SN, U202 MCP2515-xSO, U401 ATMEGA328P-PU, U501 LM7805, Y201 16MHz, Y401 16MHz

Commit message: Footprints
Parts:
- removed C1, C3, C4: 100n, Capacitor_SMD:C_0805_2012Metric_Pad1.15x1.40mm_HandSolder
- removed C2: 1n, Capacitor_SMD:C_0805_2012Metric_Pad1.15x1.40mm_HandSolder
- removed C5, C6, C7, C8: 4700u 35V, Capacitor_THT:CP_Radial_D18.0mm_P7.50mm
- removed D1, D5: G3mm, LED_SMD:LED_0805_2012Metric_Pad1.15x1.40mm_HandSolder
- removed D2: LL4148, Diode_SMD:D_MiniMELF
- removed D3: R3mm, LED_SMD:LED_0805_2012Metric_Pad1.15x1.40mm_HandSolder
- removed D4: MUR460, Diode_THT:D_DO-201AD_P15.24mm_Horizontal
- removed F1: 3A, KicadZeniteSolarLibrary18:Fuse_Holder_5x20
- removed F2: 10A, KicadZeniteSolarLibrary18:Fuse_Holder_5x20
- removed H101, H102, H103, H104: MountingHole, MountingHole:MountingHole_3.2mm_M3
- removed J1: Screw_Terminal_01x02, TerminalBlock:TerminalBlock_bornier-2_P5.08mm
- removed J2: Screw_Terminal_01x03, TerminalBlock:TerminalBlock_bornier-3_P5.08mm
- removed JP1: SolderJumper_3_Bridged12, Jumper:SolderJumper-3_P1.3mm_Bridged2Bar12_Pad1.0x1.5mm_NumberLabels
- removed K1: coil: 12VDC, contact: 125V/10A, Relay_THT:Relay_SPDT_SANYOU_SRD_Series_Form_C
- removed Q1: BCV27, Package_TO_SOT_SMD:TSOT-23_HandSoldering
- removed R1: 330R, Resistor_SMD:R_0805_2012Metric_Pad1.15x1.40mm_HandSolder
- removed R2: NC, Resistor_SMD:R_0805_2012Metric_Pad1.15x1.40mm_HandSolder
- removed R3: 1k2, Resistor_SMD:R_0805_2012Metric_Pad1.15x1.40mm_HandSolder
- removed R4, R7, R8: 1k, Resistor_SMD:R_0805_2012Metric_Pad1.15x1.40mm_HandSolder
- removed R5: 10k, Resistor_SMD:R_0805_2012Metric_Pad1.15x1.40mm_HandSolder
- removed R6: 120R, Resistor_SMD:R_0805_2012Metric_Pad1.15x1.40mm_HandSolder
- removed TP1: A1, TestPoint:TestPoint_Pad_D1.5mm
- removed TP2: K1, TestPoint:TestPoint_Pad_D1.5mm
- removed TP3: 12V, TestPoint:TestPoint_Pad_D1.5mm
- removed TP4: B1, TestPoint:TestPoint_Pad_D1.5mm
- removed TP5: OUT1, TestPoint:TestPoint_Pad_D1.5mm
- removed U1: 4N25, Package_DIP:DIP-6_W8.89mm_SMDSocket_LongPads
- added C301: 100n, Capacitor_SMD:C_0805_2012Metric_Pad1.15x1.40mm_HandSolder, B.Cu at (151.7, 40.8)
- added C302: 100n, Capacitor_SMD:C_0805_2012Metric_Pad1.15x1.40mm_HandSolder, B.Cu at (131.1, 29.1)
- added C303: 100n, Capacitor_SMD:C_0805_2012Metric_Pad1.15x1.40mm_HandSolder, B.Cu at (149.8, 35.0)
- added C304: 100n, Capacitor_SMD:C_0805_2012Metric_Pad1.15x1.40mm_HandSolder, B.Cu at (155.4, 42.8)
- added C305: 100n, Capacitor_SMD:C_0805_2012Metric_Pad1.15x1.40mm_HandSolder, B.Cu at (146.1, 31.6)
- added C306: 100n, Capacitor_SMD:C_0805_2012Metric_Pad1.15x1.40mm_HandSolder, B.Cu at (151.7, 38.9)
- added C307: 100n, Capacitor_SMD:C_0805_2012Metric_Pad1.15x1.40mm_HandSolder, B.Cu at (142.4, 27.7)
- added C308: 100n, Capacitor_SMD:C_0805_2012Metric_Pad1.15x1.40mm_HandSolder, B.Cu at (142.4, 29.7)
- added C801: 100n, Capacitor_SMD:C_0805_2012Metric_Pad1.15x1.40mm_HandSolder, B.Cu at (-10.5, 72.6)
- added C802: 100n, Capacitor_SMD:C_0805_2012Metric_Pad1.15x1.40mm_HandSolder, B.Cu at (19.5, 95.0)
- added C803: 1uF, Capacitor_SMD:C_0805_2012Metric_Pad1.15x1.40mm_HandSolder, B.Cu at (1.78, 84.6)
- added C804: 100n, Capacitor_SMD:C_0805_2012Metric_Pad1.15x1.40mm_HandSolder, B.Cu at (19.5, 87.2)
- added C805: 100nF, Capacitor_SMD:C_0805_2012Metric_Pad1.15x1.40mm_HandSolder, B.Cu at (-5.17, 77.3)
- added C806: 100n, Capacitor_SMD:C_0805_2012Metric_Pad1.15x1.40mm_HandSolder, B.Cu at (19.5, 89.2)
- added C807: 100n, Capacitor_SMD:C_0805_2012Metric_Pad1.15x1.40mm_HandSolder, B.Cu at (-55.3, 80.5)
- added C808: 100n, Capacitor_SMD:C_0805_2012Metric_Pad1.15x1.40mm_HandSolder, B.Cu at (1.78, 86.5)
- added C809: 100n, Capacitor_SMD:C_0805_2012Metric_Pad1.15x1.40mm_HandSolder, B.Cu at (-16.8, 70.0)
- added C810: 100n, Capacitor_SMD:C_0805_2012Metric_Pad1.15x1.40mm_HandSolder, B.Cu at (11.7, 96.2)
- added C811: 100nF, Capacitor_SMD:C_0805_2012Metric_Pad1.15x1.40mm_HandSolder, B.Cu at (1.78, 90.4)
- added C812: 4700u, Capacitor_SMD:C_0805_2012Metric_Pad1.15x1.40mm_HandSolder, B.Cu at (-6.72, 75.4)
- added C813: 1uF, Capacitor_Tantalum_SMD:CP_EIA-6032-20_AVX-F_Pad2.25x2.35mm_HandSolder, B.Cu at (-47.8, 69.4)
- added D301: 4V7, Diode_SMD:D_MiniMELF_Handsoldering, B.Cu at (133.9, 42.6)
- added D302: 4V7, Diode_SMD:D_MiniMELF_Handsoldering, B.Cu at (133.9, 40.4)
- added D801: LL4148, Diode_SMD:D_MiniMELF_Handsoldering, B.Cu at (-35.2, 68.4)
- added D802: LL4148, Diode_SMD:D_MiniMELF_Handsoldering, B.Cu at (19.5, 97.0)
- added D803: LL4148, Diode_SMD:D_MiniMELF_Handsoldering, B.Cu at (-12.6, 98.9)
- added D804: LL4148, Diode_SMD:D_MiniMELF_Handsoldering, B.Cu at (-40.4, 85.3)
- added D805: RED_LED, LED_SMD:LED_0805_2012Metric_Pad1.15x1.40mm_HandSolder, B.Cu at (-21.6, 90.2)
- added D806: GRN_LED, LED_SMD:LED_0805_2012Metric_Pad1.15x1.40mm_HandSolder, B.Cu at (-8.02, 99.0)
- added D807: YLW_LED, LED_SMD:LED_0805_2012Metric_Pad1.15x1.40mm_HandSolder, B.Cu at (-54.5, 68.1)
- added D808: GRN_LED, LED_SMD:LED_0805_2012Metric_Pad1.15x1.40mm_HandSolder, B.Cu at (-30.5, 69.2)
- added F801: 500mA, Fuse:Fuse_1206_3216Metric_Pad1.42x1.75mm_HandSolder, B.Cu at (-58.9, 68.0)
- added F802: Fuse Mega 200A, KicadZeniteSolarLibrary18:MegaFuse, F.Cu at (168.3, -80.6)
- added H1: MountingHole, MountingHole:MountingHole_3.2mm_M3, B.Cu at (-31.9, 73.7)
- added H2: MountingHole, MountingHole:MountingHole_3.2mm_M3, B.Cu at (-10.5, 81.0)
- added H3: MountingHole, MountingHole:MountingHole_3.2mm_M3, B.Cu at (-3.57, 87.9)
- added H301: MountingHole, MountingHole:MountingHole_3.2mm_M3, B.Cu at (-51.0, 52.9)
- added H302: MountingHole, MountingHole:MountingHole_3.2mm_M3, B.Cu at (-51.0, 59.9)
- added H303: MountingHole, MountingHole:MountingHole_3.2mm_M3, B.Cu at (-57.9, 52.9)
- added H304: MountingHole, MountingHole:MountingHole_3.2mm_M3, B.Cu at (-57.9, 59.9)
- added H4: MountingHole, MountingHole:MountingHole_3.2mm_M3, B.Cu at (-10.5, 87.9)
- added H801: U_BAT+, MountingHole:MountingHole_3.2mm_M3_DIN965_Pad, B.Cu at (-25.3, 74.1)
- added H802: +BAT, MountingHole:MountingHole_3.2mm_M3_DIN965_Pad, F.Cu at (201.3, -4.45)
- added H803: U_BAT-, MountingHole:MountingHole_3.2mm_M3_DIN965_Pad, B.Cu at (6.78, 94.1)
- added H804: F_BAT-, MountingHole:MountingHole_3.2mm_M3_DIN965_Pad, B.Cu at (-3.97, 81.4)
- added H805: MountingHole, MountingHole:MountingHole_3.2mm_M3, B.Cu at (-17.5, 80.6)
- added H806: MountingHole, MountingHole:MountingHole_3.2mm_M3, B.Cu at (-38.8, 75.2)
- added H807: MountingHole, MountingHole:MountingHole_3.2mm_M3, B.Cu at (-31.4, 80.6)
- added H808: MountingHole, MountingHole:MountingHole_3.2mm_M3, B.Cu at (-24.4, 80.6)
- added J101: Conn_01x11_Male, KicadZeniteSolarLibrary18:PinHeader_1x11_P2.54mm_Vertical_HandSoldering, F.Cu at (129.5, 61.6)
- added J102: Conn_01x11_Male, KicadZeniteSolarLibrary18:PinHeader_1x11_P2.54mm_Vertical_HandSoldering, F.Cu at (104.1, 71.8)
- added J703: RJ45, KicadZeniteSolarLibrary18:RJ45_YH59_01, F.Cu at (163.2, 125.1)
- added J704: RJ45, KicadZeniteSolarLibrary18:RJ45_YH59_01, F.Cu at (182.9, 125.7)
- added JP801: Jp_TEST, Resistor_SMD:R_0805_2012Metric_Pad1.15x1.40mm_HandSolder, B.Cu at (-13.1, 70.3)
- added JP802: Jp_TEST, Resistor_SMD:R_0805_2012Metric_Pad1.15x1.40mm_HandSolder, B.Cu at (-16.8, 68.1)
- added JP803: Jp_TEST, Resistor_SMD:R_0805_2012Metric_Pad1.15x1.40mm_HandSolder, B.Cu at (5.53, 88.1)
- added K801: DIPxx-1Axx-13x, KicadZeniteSolarLibrary18:Mega_Relay_K100, F.Cu at (119.4, -8.26)
- added K802: SANYOU_SRD_Form_C, Relay_THT:Relay_SPDT_SANYOU_SRD_Series_Form_C, F.Cu at (128.9, -57.8)
- added NT801: Net-Tie_2, Resistor_SMD:R_0805_2012Metric_Pad1.15x1.40mm_HandSolder, B.Cu at (9.28, 90.0)
- added Q801: BCV27, Package_TO_SOT_SMD:TSOT-23_HandSoldering, B.Cu at (-40.4, 95.9)
- added Q802: Q_NPN_BEC, Package_TO_SOT_SMD:TSOT-23_HandSoldering, B.Cu at (123.2, -52.7)
- added Q803: BCV27, Package_TO_SOT_SMD:TSOT-23_HandSoldering, B.Cu at (-40.9, 68.5)
- added R301: 10k, Resistor_SMD:R_0805_2012Metric_Pad1.15x1.40mm_HandSolder, B.Cu at (147.9, 40.8)
- added R302: 100k, Resistor_SMD:R_0805_2012Metric_Pad1.15x1.40mm_HandSolder, B.Cu at (134.9, 27.1)
- added R303: 10k, Resistor_SMD:R_0805_2012Metric_Pad1.15x1.40mm_HandSolder, B.Cu at (142.3, 33.6)
- added R304: 10k, Resistor_SMD:R_0805_2012Metric_Pad1.15x1.40mm_HandSolder, B.Cu at (134.9, 29.1)
- added R305: 1k, Resistor_SMD:R_0805_2012Metric_Pad1.15x1.40mm_HandSolder, B.Cu at (138.6, 31.6)
- added R306: 1k, Resistor_SMD:R_0805_2012Metric_Pad1.15x1.40mm_HandSolder, B.Cu at (131.1, 27.1)
- added R307: 1k, Resistor_SMD:R_0805_2012Metric_Pad1.15x1.40mm_HandSolder, B.Cu at (155.4, 40.8)
- added R308: 10k, Resistor_SMD:R_0805_2012Metric_Pad1.15x1.40mm_HandSolder, B.Cu at (151.7, 36.9)
- added R309: 10k, Resistor_SMD:R_0805_2012Metric_Pad1.15x1.40mm_HandSolder, B.Cu at (159.2, 42.8)
- added R310: 10k, Resistor_SMD:R_0805_2012Metric_Pad1.15x1.40mm_HandSolder, B.Cu at (147.9, 36.9)
- added R311: 100k, Resistor_SMD:R_0805_2012Metric_Pad1.15x1.40mm_HandSolder, B.Cu at (147.9, 42.8)
- added R312: 10k, Resistor_SMD:R_0805_2012Metric_Pad1.15x1.40mm_HandSolder, B.Cu at (146.1, 33.6)
- added R313: 10k, Resistor_SMD:R_0805_2012Metric_Pad1.15x1.40mm_HandSolder, B.Cu at (142.3, 31.6)
- added R314: 1k, Resistor_SMD:R_0805_2012Metric_Pad1.15x1.40mm_HandSolder, B.Cu at (138.6, 27.7)
- added R315: 1k, Resistor_SMD:R_0805_2012Metric_Pad1.15x1.40mm_HandSolder, B.Cu at (138.6, 29.7)
- added R316: 1k, Resistor_SMD:R_0805_2012Metric_Pad1.15x1.40mm_HandSolder, B.Cu at (147.9, 38.9)
- added R317: 10k, Resistor_SMD:R_0805_2012Metric_Pad1.15x1.40mm_HandSolder, B.Cu at (151.7, 42.8)
- added R318: 10k, Resistor_SMD:R_0805_2012Metric_Pad1.15x1.40mm_HandSolder, B.Cu at (138.6, 33.6)
- added R801: 1k2, Resistor_SMD:R_0805_2012Metric_Pad1.15x1.40mm_HandSolder, B.Cu at (11.7, 94.2)
- added R802: 1k2, Resistor_SMD:R_0805_2012Metric_Pad1.15x1.40mm_HandSolder, B.Cu at (19.5, 93.1)
- added R803: 10k, Resistor_SMD:R_0805_2012Metric_Pad1.15x1.40mm_HandSolder, B.Cu at (-10.5, 74.6)
- added R804: 10k, Resistor_SMD:R_0805_2012Metric_Pad1.15x1.40mm_HandSolder, B.Cu at (-20.6, 70.0)
- added R805: 120, Resistor_SMD:R_0805_2012Metric_Pad1.15x1.40mm_HandSolder, B.Cu at (-14.2, 74.2)
- added R806: 120, Resistor_SMD:R_0805_2012Metric_Pad1.15x1.40mm_HandSolder, B.Cu at (5.53, 90.0)
- added R807: 1R, Resistor_SMD:R_0805_2012Metric_Pad1.15x1.40mm_HandSolder, B.Cu at (-14.2, 72.3)
- added R808: 1R, Resistor_SMD:R_0805_2012Metric_Pad1.15x1.40mm_HandSolder, B.Cu at (-10.5, 76.5)
- added R809: 120, Resistor_SMD:R_0805_2012Metric_Pad1.15x1.40mm_HandSolder, B.Cu at (-20.6, 68.1)
- added R810: 10k, Resistor_SMD:R_0805_2012Metric_Pad1.15x1.40mm_HandSolder, B.Cu at (-14.2, 76.2)
- added R811: 1k2, Resistor_SMD:R_0805_2012Metric_Pad1.15x1.40mm_HandSolder, B.Cu at (1.78, 88.5)
- added R812: 10R, Resistor_THT:R_Axial_Power_L48.0mm_W12.5mm_P55.88mm, F.Cu at (150.5, -37.5)
- added R813: 2k5, Resistor_SMD:R_0805_2012Metric_Pad1.15x1.40mm_HandSolder, B.Cu at (19.5, 91.1)
- added R814: 2k5, Resistor_SMD:R_0805_2012Metric_Pad1.15x1.40mm_HandSolder, B.Cu at (0.98, 82.6)
- added R815: 470, Resistor_SMD:R_0805_2012Metric_Pad1.15x1.40mm_HandSolder, B.Cu at (-13.1, 68.4)
- added R816: 470, Resistor_SMD:R_0805_2012Metric_Pad1.15x1.40mm_HandSolder, B.Cu at (19.5, 85.3)
- added TH801: 60R, Resistor_THT:R_Axial_DIN0204_L3.6mm_D1.6mm_P7.62mm_Horizontal, F.Cu at (94.6, -48.3)
- added TP13: +12V, TestPoint:TestPoint_Pad_2.0x2.0mm, B.Cu at (151.9, 28.3)
- added TP301: op_a_in-, TestPoint:TestPoint_Pad_2.0x2.0mm, B.Cu at (153.2, 34.4)
- added TP302: op_a_out, TestPoint:TestPoint_Pad_2.0x2.0mm, B.Cu at (149.5, 32.5)
- added TP303: in-, TestPoint:TestPoint_Pad_2.0x2.0mm, B.Cu at (148.8, 29.1)
- added TP304: op_b_out, TestPoint:TestPoint_Pad_2.0x2.0mm, B.Cu at (152.5, 31.4)
- added TP305: op_b_in+, TestPoint:TestPoint_Pad_2.0x2.0mm, B.Cu at (158.1, 37.2)
- added TP306: in+, TestPoint:TestPoint_Pad_2.0x2.0mm, B.Cu at (155.1, 38.3)
- added TP307: op_a_in+, TestPoint:TestPoint_Pad_2.0x2.0mm, B.Cu at (145.8, 29.1)
- added TP308: op_a_in-, TestPoint:TestPoint_Pad_2.0x2.0mm, B.Cu at (156.3, 34.2)
- added TP309: op_a_out, TestPoint:TestPoint_Pad_2.0x2.0mm, B.Cu at (159.3, 34.2)
- added TP310: in-, TestPoint:TestPoint_Pad_2.0x2.0mm, B.Cu at (155.6, 31.1)
- added TP311: op_b_out, TestPoint:TestPoint_Pad_2.0x2.0mm, B.Cu at (158.6, 31.1)
- added TP312: op_b_in+, TestPoint:TestPoint_Pad_2.0x2.0mm, B.Cu at (154.9, 28.1)
- added TP313: in+, TestPoint:TestPoint_Pad_2.0x2.0mm, B.Cu at (158.0, 28.1)
- added TP314: op_a_in+, TestPoint:TestPoint_Pad_2.0x2.0mm, B.Cu at (158.8, 40.3)
- added TP801: RL_ON, TestPoint:TestPoint_Pad_D1.5mm, B.Cu at (14.9, 95.9)
- added TP802: Charge, TestPoint:TestPoint_Pad_D1.5mm, B.Cu at (12.4, 92.0)
- added TP803: B_CH, TestPoint:TestPoint_Pad_D1.5mm, B.Cu at (-7.35, 70.4)
- added TP804: B_ON, TestPoint:TestPoint_Pad_D1.5mm, B.Cu at (8.68, 87.8)
- added TP805: ON, TestPoint:TestPoint_Pad_D1.5mm, B.Cu at (-4.87, 98.8)
- added TP806: CH-, TestPoint:TestPoint_Pad_D1.5mm, B.Cu at (0.38, 80.4)
- added TP807: OFF, TestPoint:TestPoint_Pad_D1.5mm, B.Cu at (-9.90, 70.4)
- added TP808: CH+, TestPoint:TestPoint_Pad_D1.5mm, B.Cu at (13.3, 120.7)
- added TP809: B_OFF, TestPoint:TestPoint_Pad_D1.5mm, B.Cu at (-7.32, 73.1)
- added TP810: TH+, TestPoint:TestPoint_Pad_D1.5mm, B.Cu at (-2.02, 77.0)
- added TP811: TH-, TestPoint:TestPoint_Pad_D1.5mm, B.Cu at (-9.90, 67.8)
- added TP812: RL_OFF, TestPoint:TestPoint_Pad_D1.5mm, B.Cu at (4.93, 85.8)
- added U301: LM324, Package_SO:SOIC-14_3.9x8.7mm_P1.27mm, B.Cu at (133.0, 34.7)
- added U302: LM324, Package_SO:SOIC-14_3.9x8.7mm_P1.27mm, B.Cu at (142.3, 39.2)
- added U801: LM7812, Package_SO:SOIC-8_3.9x4.9mm_P1.27mm, B.Cu at (-48.7, 87.0)
- renumbered J601 to J701, J602 to J702
Connections:
- net /CANBUS CONN/CAN_H renamed /CONTROLLER/sheet5CA5A59C/CAN_H
- net /CANBUS CONN/CAN_L renamed /CONTROLLER/sheet5CA5A59C/CAN_L
- net /CANBUS/CS renamed /CONTROLLER/sheet5CA5A59C/CS
- net /CANBUS/INT renamed /CONTROLLER/sheet5CA5A59C/INT
- net /CANBUS/RXCAN renamed /CONTROLLER/sheet5CA5A59C/RXCAN
- net /CANBUS/TXCAN renamed /CONTROLLER/sheet5CA5A59C/TXCAN
- net /MCU/LED1 renamed /CONTROLLER/sheet5CA5A59D/LED1
- net /MCU/LED2 renamed /CONTROLLER/sheet5CA5A59D/LED2
- net /MCU/RESET renamed /CONTROLLER/sheet5CA5A59D/RESET
- net /MCU/USART_RX renamed /CONTROLLER/sheet5CA5A59D/USART_RX
- net /MCU/USART_TX renamed /CONTROLLER/sheet5CA5A59D/USART_TX
- net /MISO renamed /CONTROLLER/MISO
- net /MOSI renamed /CONTROLLER/MOSI
- net /POWER SUPPLY/+18V_IN renamed /CONTROLLER/+18V_OUT
- net /SCK renamed /CONTROLLER/SCK
- U401 pad 23: Net-(U401-Pad23) -> /CONTROLLER/Charge
- U401 pad 24: Net-(U401-Pad24) -> /CONTROLLER/RL_OFF
- U401 pad 25: Net-(U401-Pad25) -> /CONTROLLER/RL_ON
- U401 pad 26: Net-(U401-Pad26) -> /CONTROLLER/sig_cap+
- U401 pad 27: Net-(U401-Pad27) -> /CONTROLLER/sig_bat+
- U401 pad 4: /MCU/ON_OFF_PUMP -> Net-(U401-Pad4)
Routing:
- net GNDPWR: track 231.7 -> 0.00 mm
- net +12V: track 126.9 -> 0.00 mm
- net /pump_driver/+Pump: track 69.5 -> 0.00 mm
- net /pump_driver/Level_sensor: track 68.4 -> 0.00 mm
- net Net-(C4-Pad1): track 29.0 -> 0.00 mm
- net Net-(U401-Pad4): track 0.00 -> 23.3 mm
- net /MCU/ON_OFF_PUMP: track 23.3 -> 0.00 mm
- net Net-(JP1-Pad1): track 22.1 -> 0.00 mm
- net Net-(C3-Pad1): track 14.6 -> 0.00 mm
- net /filter/Vin: track 11.0 -> 0.00 mm
- net Net-(D2-Pad2): track 9.47 -> 0.00 mm
- net Net-(C2-Pad2): track 6.59 -> 0.00 mm
- net Net-(JP1-Pad3): track 6.18 -> 0.00 mm
- net Net-(Q1-Pad2): track 3.68 -> 0.00 mm
- net Net-(D3-Pad1): track 2.78 -> 0.00 mm
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- removed copper zone on B.Cu, net GNDPWR

Commit message: Generic layout and relay driver
Parts:
- moved D803 216.3 mm to (137.8, -56.5), turned to 90 degrees
- moved R806 206.4 mm to (144.1, -62.9), turned to 270 degrees
- moved R804 203.9 mm to (142.2, -52.7), turned to 180 degrees
- moved C802 194.1 mm to (142.2, -55.2), turned to 180 degrees
- moved R808 189.2 mm to (123.8, -56.8), turned to 180 degrees
- moved R802 188.6 mm to (143.1, -49.3), turned to 270 degrees
- moved Q801 187.4 mm to (125.1, 8.06), turned to 90 degrees
- moved C806 182.3 mm to (128.7, -56.8), turned to 180 degrees
- moved D804 174.0 mm to (113.0, 3.17), turned to 270 degrees
- moved Q803 171.8 mm to (120.0, 8.26), turned to 90 degrees
- moved R805 158.1 mm to (127.0, 3.17), turned to 270 degrees
- moved R809 155.4 mm to (120.7, 3.17), turned to 270 degrees
- moved C809 148.3 mm to (120.0, 12.7), turned to 180 degrees
- moved C801 148.2 mm to (125.1, 12.7), turned to 180 degrees
- moved R803 148.0 mm to (125.1, 15.2), turned to 180 degrees
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Connections:
- C807 pad 1: /CHARGER/+BAT -> /CHARGER/+CAP
- H802 pad 1: /CHARGER/+BAT -> /CHARGER/+CAP
- K801 pad 5: /CHARGER/+BAT -> /CHARGER/+CAP
- K802 pad 3: /CHARGER/Charge -> /CHARGER/CH
- R808 pad 2: /CHARGER/Charge -> /CHARGER/CH
- TH801 pad 2: /CHARGER/Charge -> /CHARGER/CH
- TP810 pad 1: /CHARGER/Charge -> /CHARGER/CH
Routing:
- net GNDPWR: track 0.00 -> 168.4 mm
- net /CHARGER/+12V: track 0.00 -> 72.7 mm
- net /CHARGER/Charge: track 0.00 -> 55.0 mm
- net /CHARGER/U_BAT+: track 0.00 -> 51.0 mm
- net /CHARGER/CH: track 0.00 -> 27.4 mm
- net Net-(R812-Pad2): track 0.00 -> 25.4 mm
- net /CHARGER/+CAP: track 0.00 -> 19.1 mm
- net Net-(D802-Pad2): track 0.00 -> 18.0 mm
- net Net-(D803-Pad2): track 0.00 -> 17.5 mm
- net Net-(D804-Pad2): track 0.00 -> 9.85 mm
- net Net-(C801-Pad1): track 0.00 -> 7.89 mm
- net Net-(C809-Pad1): track 0.00 -> 7.72 mm
- net Net-(C802-Pad1): track 0.00 -> 7.69 mm
- net Net-(K801-Pad2): track 0.00 -> 4.85 mm
- net Net-(K801-Pad3): track 0.00 -> 4.37 mm
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Other:
- net class Default: trace_width 0.508 -> 0.762
- board text added: "Copper Bar"

Commit message: Copper bar fixation
Parts:
- removed C308: 100n, Capacitor_SMD:C_0805_2012Metric_Pad1.15x1.40mm_HandSolder
- removed C803: 1uF, Capacitor_SMD:C_0805_2012Metric_Pad1.15x1.40mm_HandSolder
- removed C805, C811: 100nF, Capacitor_SMD:C_0805_2012Metric_Pad1.15x1.40mm_HandSolder
- removed C813: 1uF, Capacitor_Tantalum_SMD:CP_EIA-6032-20_AVX-F_Pad2.25x2.35mm_HandSolder
- removed D801: LL4148, Diode_SMD:D_MiniMELF_Handsoldering
- removed F801: 500mA, Fuse:Fuse_1206_3216Metric_Pad1.42x1.75mm_HandSolder
- removed U302: LM324, Package_SO:SOIC-14_3.9x8.7mm_P1.27mm
- removed U801: LM7812, Package_SO:SOIC-8_3.9x4.9mm_P1.27mm
- added C1: 1uF, Capacitor_SMD:C_0805_2012Metric_Pad1.15x1.40mm_HandSolder, B.Cu at (-28.3, 41.8)
- added C2: 100nF, Capacitor_SMD:C_0805_2012Metric_Pad1.15x1.40mm_HandSolder, B.Cu at (-31.3, 39.9)
- added C3: 100nF, Capacitor_SMD:C_0805_2012Metric_Pad1.15x1.40mm_HandSolder, B.Cu at (-27.5, 39.9)
- added C4: 1uF, Capacitor_Tantalum_SMD:CP_EIA-6032-20_AVX-F_Pad2.25x2.35mm_HandSolder, B.Cu at (-34.1, 44.1)
- added D1: LL4148, Diode_SMD:D_MiniMELF_Handsoldering, B.Cu at (-33.4, 47.1)
- added F1: 500mA, Fuse:Fuse_1206_3216Metric_Pad1.42x1.75mm_HandSolder, B.Cu at (-35.6, 41.1)
- added U1: LM7812, Package_SO:SOIC-8_3.9x4.9mm_P1.27mm, B.Cu at (-25.0, 45.5)
- C812: footprint Capacitor_SMD:C_0805_2012Metric_Pad1.15x1.40mm_HandSolder -> Capacitor_THT:CP_Radial_D10.0mm_P5.00mm; moved to F.Cu
- moved JP802 295.2 mm to (253.4, -50.8)
- moved H807 270.1 mm to (188.0, -77.1)
- moved H303 256.9 mm to (188.0, -21.6)
- moved H805 250.8 mm to (177.6, -77.1)
- moved H804 233.5 mm to (167.6, -77.1)
- moved H3 228.4 mm to (178.6, -49.8)
- moved H808 226.4 mm to (177.6, -21.6)
- moved H1 216.1 mm to (122.6, -77.5)
- moved H301 210.7 mm to (130.2, -54.6)
- moved JP801 200.2 mm to (135.3, -64.1), turned to 270 degrees
- moved TP806 187.0 mm to (117.5, -65.4)
- moved H803 186.2 mm to (78.1, -77.9)
- moved C810 181.4 mm to (119.8, -49.5)
- moved H4 179.8 mm to (59.1, -77.9)
- moved H2 177.5 mm to (68.8, -77.9)
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Connections:
- U301 pad 1: (no net) -> Net-(R301-Pad1)
- U301 pad 10: Net-(R308-Pad1) -> Net-(R317-Pad1)
- U301 pad 12: (no net) -> Net-(C307-Pad1)
- U301 pad 13: (no net) -> /CHARGER/sig_cap+
- U301 pad 14: (no net) -> /CHARGER/sig_cap+
- U301 pad 2: (no net) -> Net-(R301-Pad2)
- U301 pad 3: (no net) -> Net-(R308-Pad1)
- U301 pad 8: Net-(R301-Pad1) -> Net-(R310-Pad1)
- U301 pad 9: Net-(R301-Pad2) -> Net-(R310-Pad2)
Routing:
- net GNDPWR: track 168.4 -> 89.7 mm
- net /CHARGER/+12V: track 72.7 -> 137.2 mm
- net Net-(R812-Pad2): track 25.4 -> 9.79 mm
- net /CHARGER/Charge: track 55.0 -> 39.5 mm
- net /CHARGER/U_BAT+: track 51.0 -> 37.7 mm
- net Net-(D802-Pad2): track 18.0 -> 6.15 mm
- net Net-(K801-Pad3): track 4.37 -> 11.7 mm
- net Net-(K801-Pad2): track 4.85 -> 11.9 mm
- net Net-(D803-Pad2): track 17.5 -> 22.8 mm
- net /CHARGER/RL_OFF: track 0.00 -> 3.01 mm
- net /CHARGER/RL_ON: track 0.00 -> 2.91 mm
- net Net-(C809-Pad1): track 7.72 -> 10.5 mm
- net Net-(C801-Pad1): track 7.89 -> 10.3 mm
- net /CHARGER/CH: track 27.4 -> 25.4 mm
- net Net-(D804-Pad2): track 9.85 -> 8.22 mm

Commit message: Layout and Relay footprint
Parts:
- removed J101, J102: Conn_01x11_Male, KicadZeniteSolarLibrary18:PinHeader_1x11_P2.54mm_Vertical_HandSoldering
- removed K801: DIPxx-1Axx-13x, KicadZeniteSolarLibrary18:Mega_Relay_K100
- added J1: Conn_02x11_Odd_Even, KicadZeniteSolarLibrary18:PinHeader_2x11_P2.54mm_Vertical_HandSoldering, B.Cu at (144.8, 12.1)
- added J2: Conn_02x11_Odd_Even, KicadZeniteSolarLibrary18:PinHeader_2x11_P2.54mm_Vertical_HandSoldering, F.Cu at (130.2, 69.2)
- added K1: K100A, Connector_PinHeader_2.54mm:PinHeader_1x03_P2.54mm_Vertical_SMD_Pin1Right, B.Cu at (81.4, 3.13)
- added U2: K100B, KicadZeniteSolarLibrary18:Mega_Relay_K100_separated, F.Cu at (119.4, -8.26)
- F802: moved to B.Cu
- U1: footprint Package_SO:SOIC-8_3.9x4.9mm_P1.27mm -> KicadZeniteSolarLibrary18:TO-220-3_Horizontal_TabDown_SMD
- moved C4 207.0 mm to (166.8, -5.49), turned to 180 degrees
- moved C3 200.8 mm to (168.7, -2.32), turned to 180 degrees
- moved C2 196.8 mm to (160.5, -4.22)
- moved F1 195.3 mm to (154.3, -4.45), turned to 90 degrees
- moved C1 194.8 mm to (160.5, -6.13)
- moved D1 192.7 mm to (154.3, 3.81), turned to 270 degrees
- moved U1 190.2 mm to (159.9, 0.86)
- moved R815 30.1 mm to (-38.7, 52.7)
- moved D804 14.1 mm to (89.0, -4.49)
- moved Q801 14.1 mm to (92.2, 7.57)
- moved Q803 14.1 mm to (92.2, 0.59)
- moved R805 14.1 mm to (87.1, 5.67)
- moved R809 14.1 mm to (87.1, -0.05)
- moved TP801 14.1 mm to (103.4, 3.76)
- moved C801 14.1 mm to (96.6, 7.57)
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Routing:
- net /CHARGER/+12V: track 137.2 -> 266.8 mm
- net GNDPWR: track 89.7 -> 157.6 mm
- net /CHARGER/+18V_IN: track 0.00 -> 13.9 mm
- net Net-(C1-Pad1): track 23.9 -> 11.5 mm
- net Net-(D1-Pad1): track 0.00 -> 4.02 mm
- net Net-(K1-Pad1): track 11.7 -> 10.4 mm
- net Net-(K1-Pad3): track 11.9 -> 10.7 mm
- net /CHARGER/RL_OFF: track 3.01 -> 3.69 mm
- net /CHARGER/RL_ON: track 2.91 -> 3.59 mm

Commit message: Ampop layout not finished
Parts:
- moved NT801 200.6 mm to (132.1, -68.6)
- moved TP803 186.2 mm to (129.5, -55.9)
- moved TP802 184.6 mm to (129.5, -50.8)
- moved JP803 174.4 mm to (150.5, -8.89), turned to 180 degrees
- moved TP810 168.2 mm to (91.4, -62.9)
- moved TP811 152.7 mm to (83.8, -52.7)
- moved R309 133.5 mm to (137.7, -62.9)
- moved R311 128.5 mm to (131.9, -46.4), turned to 180 degrees
- moved R317 127.9 mm to (135.8, -46.4), turned to 180 degrees
- moved R308 127.8 mm to (135.7, -64.8), turned to 180 degrees
- moved JP802 123.5 mm to (129.9, -48.3)
- moved R313 121.6 mm to (133.8, -48.3), turned to 180 degrees
- moved D301 119.2 mm to (139.7, -0.64), turned to 90 degrees
- moved R312 117.3 mm to (141.6, -48.3), turned to 180 degrees
- moved R310 117.1 mm to (143.5, -46.4), turned to 180 degrees
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Connections:
- J1 pad 11: /CHARGER/RL_OFF -> /CHARGER/Charge
- J1 pad 12: /CHARGER/RL_OFF -> /CHARGER/Charge
- J1 pad 15: /CHARGER/sig_bat+ -> /CHARGER/RL_OFF
- J1 pad 16: /CHARGER/sig_bat+ -> /CHARGER/RL_OFF
- J1 pad 19: /CHARGER/sig_cap+ -> /CHARGER/RL_ON
- J1 pad 20: /CHARGER/sig_cap+ -> /CHARGER/RL_ON
- J1 pad 3: /CHARGER/Charge -> /CHARGER/sig_bat+
- J1 pad 4: /CHARGER/Charge -> /CHARGER/sig_bat+
- J1 pad 7: /CHARGER/RL_ON -> /CHARGER/sig_cap+
- J1 pad 8: /CHARGER/RL_ON -> /CHARGER/sig_cap+
- J2 pad 11: /CONTROLLER/RL_OFF -> /CONTROLLER/Charge
- J2 pad 12: /CONTROLLER/RL_OFF -> /CONTROLLER/Charge
- J2 pad 15: /CONTROLLER/sig_bat+ -> /CONTROLLER/RL_OFF
- J2 pad 16: /CONTROLLER/sig_bat+ -> /CONTROLLER/RL_OFF
- J2 pad 19: /CONTROLLER/sig_cap+ -> /CONTROLLER/RL_ON
- J2 pad 20: /CONTROLLER/sig_cap+ -> /CONTROLLER/RL_ON
- J2 pad 3: /CONTROLLER/Charge -> /CONTROLLER/sig_bat+
- J2 pad 4: /CONTROLLER/Charge -> /CONTROLLER/sig_bat+
- J2 pad 7: /CONTROLLER/RL_ON -> /CONTROLLER/sig_cap+
- J2 pad 8: /CONTROLLER/RL_ON -> /CONTROLLER/sig_cap+
- U1 pad : GNDPWR -> (no net)
- U301 pad 1: Net-(R301-Pad1) -> Net-(R310-Pad1)
- U301 pad 10: Net-(R317-Pad1) -> Net-(C303-Pad1)
- U301 pad 2: Net-(R301-Pad2) -> Net-(R310-Pad2)
- U301 pad 3: Net-(R308-Pad1) -> Net-(R317-Pad1)
- U301 pad 5: Net-(C303-Pad1) -> Net-(R308-Pad1)
- U301 pad 6: /CHARGER/sig_bat+ -> Net-(R301-Pad2)
- U301 pad 7: /CHARGER/sig_bat+ -> Net-(R301-Pad1)
- U301 pad 8: Net-(R310-Pad1) -> /CHARGER/sig_bat+
- U301 pad 9: Net-(R310-Pad2) -> /CHARGER/sig_bat+
Routing:
- net GNDPWR: track 157.6 -> 249.5 mm
- net +12VA: track 0.00 -> 77.2 mm, vias 0 -> 2
- net /CHARGER/U_BAT+: track 37.7 -> 77.2 mm
- net /CHARGER/Charge: track 39.5 -> 72.9 mm
- net /CHARGER/RL_OFF: track 3.69 -> 34.3 mm
- net /CHARGER/+CAP: track 19.1 -> 43.2 mm, vias 0 -> 2
- net /CHARGER/RL_ON: track 3.59 -> 26.3 mm
- net /CHARGER/sig_cap+: track 0.00 -> 20.0 mm
- net /CHARGER/+12V: track 266.8 -> 286.6 mm
- net GNDA: track 0.00 -> 19.4 mm, vias 0 -> 2
- net /CHARGER/sig_bat+: track 0.00 -> 17.4 mm
- net Net-(C307-Pad1): track 0.00 -> 16.5 mm
- net Net-(R317-Pad1): track 0.00 -> 14.1 mm
- net Net-(R308-Pad1): track 0.00 -> 13.6 mm
- net Net-(R311-Pad1): track 0.00 -> 13.3 mm
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
Commit message: Circuito ampop incompleto
Parts:
- removed TP13: +12V, TestPoint:TestPoint_Pad_2.0x2.0mm
- removed TP301, TP308: op_a_in-, TestPoint:TestPoint_Pad_2.0x2.0mm
- removed TP302, TP309: op_a_out, TestPoint:TestPoint_Pad_2.0x2.0mm
- removed TP303, TP310: in-, TestPoint:TestPoint_Pad_2.0x2.0mm
- removed TP304, TP311: op_b_out, TestPoint:TestPoint_Pad_2.0x2.0mm
- removed TP305, TP312: op_b_in+, TestPoint:TestPoint_Pad_2.0x2.0mm
- removed TP306, TP313: in+, TestPoint:TestPoint_Pad_2.0x2.0mm
- removed TP307, TP314: op_a_in+, TestPoint:TestPoint_Pad_2.0x2.0mm
- TP201, TP202, TP203, TP204, TP205, TP206, TP207, TP208, TP209: footprint TestPoint:TestPoint_Pad_2.0x2.0mm -> TestPoint:TestPoint_Pad_D1.5mm
- moved H301 151.2 mm to (286.4, -40.6), turned to 90 degrees
- moved R311 117.9 mm to (249.6, -40.0), turned to 270 degrees
- moved JP802 117.4 mm to (247.0, -40.0), turned to 90 degrees
- moved R318 115.9 mm to (253.4, -41.3), turned to 90 degrees
- moved R313 113.3 mm to (247.0, -43.8), turned to 90 degrees
- moved R317 109.4 mm to (245.1, -41.9), turned to 90 degrees
- moved R312 103.5 mm to (245.1, -46.4), turned to 270 degrees
- moved R310 101.7 mm to (245.1, -50.2), turned to 270 degrees
- moved JP801 101.4 mm to (228.6, -40.0), turned to 90 degrees
- moved R309 100.1 mm to (234.9, -39.4), turned to 90 degrees
- moved R314 98.9 mm to (247.7, -62.9), turned to 0 degrees
- moved R302 97.5 mm to (226.1, -40.0), turned to 270 degrees
- moved R308 97.4 mm to (230.5, -42.5), turned to 90 degrees
- moved R304 96.6 mm to (228.6, -44.5), turned to 90 degrees
- moved C305 95.8 mm to (245.7, -64.8), turned to 180 degrees
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Routing:
- net /CHARGER/sig_cap+: track 20.0 -> 78.8 mm
- net GNDA: track 19.4 -> 0.00 mm, vias 2 -> 0
- net /CHARGER/sig_bat+: track 17.4 -> 0.00 mm
- net GNDPWR: track 249.5 -> 266.5 mm
- net Net-(C303-Pad1): track 13.2 -> 0.00 mm
- net +12VA: track 77.2 -> 64.0 mm, vias 2 -> 0
- net /CHARGER/+CAP: track 43.2 -> 35.5 mm, vias 2 -> 1
- net /CHARGER/U_BAT+: track 77.2 -> 69.8 mm
- net Net-(R302-Pad1): track 12.9 -> 5.97 mm
- net Net-(R310-Pad1): track 10.8 -> 17.3 mm, vias 0 -> 2
- net Net-(R311-Pad1): track 13.3 -> 6.95 mm
- net /CHARGER/sheet5CBAED96/in2+: track 8.22 -> 3.73 mm
- net Net-(C307-Pad1): track 16.5 -> 12.1 mm
- net /CHARGER/sheet5CBAED96/in1+: track 6.68 -> 2.39 mm
- net Net-(C301-Pad1): track 3.73 -> 0.00 mm
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