File: hardware/main/_saved_Charger.sch (KiCad schematic (older format))
At the start: 68 parts, among them K1 K100A, K802 SANYOU_SRD_Form_C, Q801 BCV27, Q802 Q_NPN_BEC, Q803 BCV27, U2 K100B

Commit message: First version PCB
Parts:
- added LOGO1: Zenite, KicadZeniteSolarLibrary18:zenite, symbol Graphic:Logo_Open_Hardware_Small
- added LOGO2: Logo_Open_Hardware_Small, Symbol:OSHW-Logo2_9.8x8mm_Copper, symbol Graphic:Logo_Open_Hardware_Small
Changed lines of the file:
@@
 NoConn ~ 6300 11300
 $Comp
-L Graphic:Logo_Open_Hardware_Small #LOGO?
+L Graphic:Logo_Open_Hardware_Small LOGO2
 U 1 1 5CC3B73E
 P 10700 8800
-F 0 "#LOGO?" H 10700 9075 50  0001 C CNN
+F 0 "LOGO2" H 10700 9075 50  0001 C CNN
 F 1 "Logo_Open_Hardware_Small" H 10700 8575 50  0001 C CNN
 F 2 "Symbol:OSHW-Logo2_9.8x8mm_Copper" H 10700 8800 50  0001 C CNN
@@
 $EndComp
 $Comp
-L Graphic:Logo_Open_Hardware_Small #LOGO1
+L Graphic:Logo_Open_Hardware_Small LOGO1
 U 1 1 5CC3C3FD
 P 10700 8150
-F 0 "#LOGO1" H 10700 8425 50  0001 C CNN
+F 0 "LOGO1" H 10700 8425 50  0001 C CNN
 F 1 "Zenite" H 10700 7925 50  0001 C CNN
 F 2 "KicadZeniteSolarLibrary18:zenite" H 10700 8150 50  0001 C CNN
