File: hardware/main/atmega328p.sch (KiCad schematic (older format))
At the start: 17 parts, among them J401 USART, U401 ATMEGA328P-PU, Y401 16MHz

Commit message: Layout retrabalhado. Não finalizado.
Connections:
- net BAT_SIG: now also U401.24 (PC1); no longer U401.27 (PC4)
- net CAP_SIG: now also U401.23 (PC0); no longer U401.26 (PC3)
- net Charge: now also U401.25 (PC2); no longer U401.23 (PC0)
- net RL_OFF: now also U401.26 (PC3); no longer U401.24 (PC1)
- net RL_ON: now also U401.27 (PC4); no longer U401.25 (PC2)
Changed lines of the file:
@@
 EESchema Schematic File Version 4
 LIBS:main-cache
-EELAYER 26 0
+EELAYER 29 0
 EELAYER END
 $Descr A4 11693 8268
@@
 Wire Wire Line
 	4950 4650 5050 4650
+Text HLabel 5050 3950 2    50   Input ~ 0
+RL_OFF
+Text HLabel 5050 4050 2    50   Input ~ 0
+RL_ON
+Text HLabel 5050 3650 2    50   Input ~ 0
+CAP_SIG
 Text HLabel 5050 3750 2    50   Input ~ 0
-RL_OFF
-Text HLabel 5050 3850 2    50   Input ~ 0
-RL_ON
-Text HLabel 5050 3950 2    50   Input ~ 0
-CAP_SIG
-Text HLabel 5050 4050 2    50   Input ~ 0
 BAT_SIG
 NoConn ~ 5050 4150
-Text HLabel 5050 3650 2    50   Input ~ 0
+Text HLabel 5050 3850 2    50   Input ~ 0
 Charge
 $EndSCHEMATC

Commit message: small update
Parts:
- J401: footprint Connector_PinHeader_2.54mm:PinHeader_1x04_P2.54mm_Vertical -> Connector_PinHeader_2.54mm:PinHeader_1x04_P2.54mm_Vertical_SMD_Pin1Left
Changed lines of the file:
@@
 F 0 "J401" H 7700 4000 50  0000 C CNN
 F 1 "USART" H 7700 4100 50  0000 C CNN
-F 2 "Connector_PinHeader_2.54mm:PinHeader_1x04_P2.54mm_Vertical" H 7750 4450 50  0001 C CNN
+F 2 "Connector_PinHeader_2.54mm:PinHeader_1x04_P2.54mm_Vertical_SMD_Pin1Left" H 7750 4450 50  0001 C CNN
 F 3 "~" H 7750 4450 50  0001 C CNN
 	1    7750 4450
